Commit message: updated the rrr_robot

File: src/robocon_description/models/rrr_robot/rrr_robot.urdf.xacro (robot description, xacro)
@@ -1,6 +1,9 @@
 <?xml version="1.0"?>
 <robot xmlns:xacro="http://www.ros.org/wiki/xacro" name="rrr_robot">
-  <xacro:property name="link_len" value="0.4"/>
-  <xacro:property name="link_rad" value="0.05"/>
+  <xacro:property name="link1_len" value="0.2"/>
+  <xacro:property name="link1b_len" value="2.7"/>
+  <xacro:property name="link2_len" value="2.7"/>
+  <xacro:property name="link3_len" value="3.5"/>
+  <xacro:property name="link_rad" value="0.2"/>
   <material name="blue"><color rgba="0 0 0.8 1"/></material>
   <material name="green"><color rgba="0 0.8 0 1"/></material>
@@ -22,13 +25,27 @@
   <link name="link1">
     <visual>
-      <origin xyz="0 0 ${link_len/2}" rpy="0 0 0"/>
-      <geometry><cylinder length="${link_len}" radius="${link_rad}"/></geometry>
+      <origin xyz="0 0 ${link1_len/2}" rpy="0 0 0"/>
+      <geometry><cylinder length="${link1_len}" radius="${link_rad}"/></geometry>
+      <material name="blue"/>
+    </visual>
+  </link>
+  <joint name="joint_new" type="revolute">
+    <parent link="link1"/>
+    <child link="link1_b"/>
+    <origin xyz="0 0 ${link1_len}" rpy="0 0 0"/>
+    <axis xyz="0 1 0"/>
+    <limit lower="-2.5" upper="2.5" effort="10.0" velocity="1.0"/>
+  </joint>
+  <link name="link1_b">
+    <visual>
+      <origin xyz="0 0 ${link1b_len/2}" rpy="0 0 0"/>
+      <geometry><cylinder length="${link1b_len}" radius="${link_rad}"/></geometry>
       <material name="blue"/>
     </visual>
   </link>
   <joint name="joint2" type="revolute">
-    <parent link="link1"/>
+    <parent link="link1_b"/>
     <child link="link2"/>
-    <origin xyz="0 0 ${link_len}" rpy="0 0 0"/>
+    <origin xyz="0 0 ${link1b_len}" rpy="0 0 0"/>
     <axis xyz="0 1 0"/>
     <limit lower="-2.5" upper="2.5" effort="10.0" velocity="1.0"/>
@@ -36,6 +53,6 @@
   <link name="link2">
     <visual>
-      <origin xyz="0 0 ${link_len/2}" rpy="0 0 0"/>
-      <geometry><cylinder length="${link_len}" radius="${link_rad*0.8}"/></geometry>
+      <origin xyz="0 0 ${link2_len/2}" rpy="0 0 0"/>
+      <geometry><cylinder length="${link2_len}" radius="${link_rad}"/></geometry>
       <material name="green"/>
     </visual>
@@ -44,5 +61,5 @@
     <parent link="link2"/>
     <child link="link3"/>
-    <origin xyz="0 0 ${link_len}" rpy="0 0 0"/>
+    <origin xyz="0 0 ${link2_len}" rpy="0 0 0"/>
     <axis xyz="0 1 0"/>
     <limit lower="-2.5" upper="2.5" effort="10.0" velocity="1.0"/>
@@ -50,8 +67,55 @@
   <link name="link3">
     <visual>
-      <origin xyz="0 0 ${link_len/2}" rpy="0 0 0"/>
-      <geometry><cylinder length="${link_len}" radius="${link_rad*0.6}"/></geometry>
+      <origin xyz="0 0 ${link3_len/2}" rpy="0 0 0"/>
+      <geometry><cylinder length="${link3_len}" radius="${link_rad}"/></geometry>
       <material name="red"/>
     </visual>
   </link>
+  <!-- Gripper Base -->
+  <!-- Gripper Base (Wrist Roll Joint) -->
+  <joint name="joint4" type="revolute">
+    <parent link="link3"/>
+    <child link="gripper_base"/>
+    <origin xyz="0 0 ${link3_len}" rpy="0 0 0"/>
+    <axis xyz="0 0 1"/>
+    <limit lower="-3.14" upper="3.14" effort="10.0" velocity="1.0"/>
+  </joint>
+  <link name="gripper_base">
+    <visual>
+      <origin xyz="0 0 0.1" rpy="0 0 0"/>
+      <geometry><box size="0.2 3 0.2"/></geometry>
+      <material name="grey"/>
+    </visual>
+  </link>
+  <!-- Left Finger -->
+  <joint name="finger_left_joint" type="prismatic">
+    <parent link="gripper_base"/>
+    <child link="gripper_finger_left"/>
+    <origin xyz="0 1.0 0.3" rpy="0 0 0"/>
+    <axis xyz="0 1 0"/>
+    <limit lower="-0.9" upper="0.5" effort="10.0" velocity="0.5"/>
+  </joint>
+  <link name="gripper_finger_left">
+    <visual>
+      <origin xyz="0 0 0" rpy="0 0 0"/>
+      <geometry><box size="0.1 0.1 0.4"/></geometry>
+      <material name="blue"/>
+    </visual>
+  </link>
+  <!-- Right Finger -->
+  <joint name="finger_right_joint" type="prismatic">
+    <parent link="gripper_base"/>
+    <child link="gripper_finger_right"/>
+    <origin xyz="0 -1.0 0.3" rpy="0 0 0"/>
+    <axis xyz="0 -1 0"/>
+    <limit lower="-1.0" upper="0.5" effort="10.0" velocity="0.5"/>
+    <mimic joint="finger_left_joint" multiplier="1.0" offset="0.0"/>
+  </joint>
+  <link name="gripper_finger_right">
+    <visual>
+      <origin xyz="0 0 0" rpy="0 0 0"/>
+      <geometry><box size="0.1 0.1 0.4"/></geometry>
+      <material name="blue"/>
+    </visual>
+  </link>
 </robot>

Commit message: better naming convention

File: src/robocon_description/models/rrr_robot/rrr_robot.urdf.xacro (robot description, xacro)
@@ -1,6 +1,6 @@
 <?xml version="1.0"?>
 <robot xmlns:xacro="http://www.ros.org/wiki/xacro" name="rrr_robot">
-  <xacro:property name="link1_len" value="0.2"/>
-  <xacro:property name="link1b_len" value="2.7"/>
+  <xacro:property name="link0_len" value="0.2"/>
+  <xacro:property name="link1_len" value="2.7"/>
   <xacro:property name="link2_len" value="2.7"/>
   <xacro:property name="link3_len" value="3.5"/>
@@ -16,10 +16,24 @@
     </visual>
   </link>
-  <joint name="joint1" type="revolute">
+  <joint name="joint0" type="revolute">
     <parent link="base_link"/>
-    <child link="link1"/>
+    <child link="link0"/>
     <origin xyz="0 0 0.05" rpy="0 0 0"/>
     <axis xyz="0 0 1"/>
     <limit lower="-3.14" upper="3.14" effort="10.0" velocity="1.0"/>
+  </joint>
+  <link name="link0">
+    <visual>
+      <origin xyz="0 0 ${link0_len/2}" rpy="0 0 0"/>
+      <geometry><cylinder length="${link0_len}" radius="${link_rad}"/></geometry>
+      <material name="blue"/>
+    </visual>
+  </link>
+  <joint name="joint1" type="revolute">
+    <parent link="link0"/>
+    <child link="link1"/>
+    <origin xyz="0 0 ${link0_len}" rpy="0 0 0"/>
+    <axis xyz="0 1 0"/>
+    <limit lower="-2.5" upper="2.5" effort="10.0" velocity="1.0"/>
   </joint>
   <link name="link1">
@@ -30,22 +44,8 @@
     </visual>
   </link>
-  <joint name="joint_new" type="revolute">
+  <joint name="joint2" type="revolute">
     <parent link="link1"/>
-    <child link="link1_b"/>
+    <child link="link2"/>
     <origin xyz="0 0 ${link1_len}" rpy="0 0 0"/>
-    <axis xyz="0 1 0"/>
-    <limit lower="-2.5" upper="2.5" effort="10.0" velocity="1.0"/>
-  </joint>
-  <link name="link1_b">
-    <visual>
-      <origin xyz="0 0 ${link1b_len/2}" rpy="0 0 0"/>
-      <geometry><cylinder length="${link1b_len}" radius="${link_rad}"/></geometry>
-      <material name="blue"/>
-    </visual>
-  </link>
-  <joint name="joint2" type="revolute">
-    <parent link="link1_b"/>
-    <child link="link2"/>
-    <origin xyz="0 0 ${link1b_len}" rpy="0 0 0"/>
     <axis xyz="0 1 0"/>
     <limit lower="-2.5" upper="2.5" effort="10.0" velocity="1.0"/>

Commit message: robot-arm attached

File: src/robocon_description/models/rrr_robot/rrr_robot.urdf.xacro (robot description, xacro)
@@ -1,18 +1,37 @@
 <?xml version="1.0"?>
 <robot xmlns:xacro="http://www.ros.org/wiki/xacro" name="rrr_robot">
-  <xacro:property name="link0_len" value="0.2"/>
-  <xacro:property name="link1_len" value="2.7"/>
-  <xacro:property name="link2_len" value="2.7"/>
-  <xacro:property name="link3_len" value="3.5"/>
-  <xacro:property name="link_rad" value="0.2"/>
+  <!--PROPERTIES -->
+  <xacro:property name="link0_len" value="0.02"/>
+  <xacro:property name="link1_len" value="0.27"/>
+  <xacro:property name="link2_len" value="0.27"/>
+  <xacro:property name="link3_len" value="0.55"/>
+  <xacro:property name="link_rad" value="0.02"/>
+  <!--  MATERIALS -->
   <material name="blue"><color rgba="0 0 0.8 1"/></material>
   <material name="green"><color rgba="0 0.8 0 1"/></material>
   <material name="red"><color rgba="0.8 0 0 1"/></material>
   <material name="grey"><color rgba="0.2 0.2 0.2 1"/></material>
+  <!--  INERTIAL MACRO  -->
+  <xacro:macro name="simple_inertial" params="mass">
+    <inertial>
+      <origin xyz="0 0 0" rpy="0 0 0"/>
+      <mass value="${mass}"/>
+      <inertia
+        ixx="${mass * 0.01}" ixy="0" ixz="0"
+        iyy="${mass * 0.01}" iyz="0"
+        izz="${mass * 0.01}"/>
+    </inertial>
+  </xacro:macro>
+  <!-- BASE -->
   <link name="base_link">
+    <xacro:simple_inertial mass="5.0"/>
     <visual>
-      <geometry><cylinder length="0.1" radius="0.15"/></geometry>
+      <geometry><cylinder length="0.05" radius="0.01"/></geometry>
       <material name="grey"/>
     </visual>
+    <collision>
+      <geometry><cylinder length="0.05" radius="0.01"/></geometry>
+      <self_collide>true</self_collide>
+    </collision>
   </link>
   <joint name="joint0" type="revolute">
@@ -23,5 +42,7 @@
     <limit lower="-3.14" upper="3.14" effort="10.0" velocity="1.0"/>
   </joint>
+  <!--  LINK 0 -->
   <link name="link0">
+    <xacro:simple_inertial mass="3.0"/>
     <visual>
       <origin xyz="0 0 ${link0_len/2}" rpy="0 0 0"/>
@@ -29,4 +50,9 @@
       <material name="blue"/>
     </visual>
+    <collision>
+      <origin xyz="0 0 ${link0_len/2}" rpy="0 0 0"/>
+      <geometry><cylinder length="${link0_len}" radius="${link_rad}"/></geometry>
+      <self_collide>true</self_collide>
+    </collision>
   </link>
   <joint name="joint1" type="revolute">
@@ -35,7 +61,9 @@
     <origin xyz="0 0 ${link0_len}" rpy="0 0 0"/>
     <axis xyz="0 1 0"/>
-    <limit lower="-2.5" upper="2.5" effort="10.0" velocity="1.0"/>
+    <limit lower="-1.57" upper="1.57" effort="10.0" velocity="1.0"/>
   </joint>
+  <!-- LINK 1 -->
   <link name="link1">
+    <xacro:simple_inertial mass="4.0"/>
     <visual>
       <origin xyz="0 0 ${link1_len/2}" rpy="0 0 0"/>
@@ -43,4 +71,9 @@
       <material name="blue"/>
     </visual>
+    <collision>
+      <origin xyz="0 0 ${link1_len/2}" rpy="0 0 0"/>
+      <geometry><cylinder length="${link1_len}" radius="${link_rad}"/></geometry>
+      <self_collide>true</self_collide>
+    </collision>
   </link>
   <joint name="joint2" type="revolute">
@@ -51,5 +84,7 @@
     <limit lower="-2.5" upper="2.5" effort="10.0" velocity="1.0"/>
   </joint>
+  <!--  LINK 2 -->
   <link name="link2">
+    <xacro:simple_inertial mass="3.5"/>
     <visual>
       <origin xyz="0 0 ${link2_len/2}" rpy="0 0 0"/>
@@ -57,4 +92,9 @@
       <material name="green"/>
     </visual>
+    <collision>
+      <origin xyz="0 0 ${link2_len/2}" rpy="0 0 0"/>
+      <geometry><cylinder length="${link2_len}" radius="${link_rad}"/></geometry>
+      <self_collide>true</self_collide>
+    </collision>
   </link>
   <joint name="joint3" type="revolute">
@@ -65,5 +105,7 @@
     <limit lower="-2.5" upper="2.5" effort="10.0" velocity="1.0"/>
   </joint>
+  <!--  LINK 3 -->
   <link name="link3">
+    <xacro:simple_inertial mass="2.5"/>
     <visual>
       <origin xyz="0 0 ${link3_len/2}" rpy="0 0 0"/>
@@ -71,7 +113,11 @@
       <material name="red"/>
     </visual>
+    <collision>
+      <origin xyz="0 0 ${link3_len/2}" rpy="0 0 0"/>
+      <geometry><cylinder length="${link3_len}" radius="${link_rad}"/></geometry>
+      <self_collide>true</self_collide>
+    </collision>
   </link>
-  <!-- Gripper Base -->
-  <!-- Gripper Base (Wrist Roll Joint) -->
+  <!-- GRIPPER BASE-->
   <joint name="joint4" type="revolute">
     <parent link="link3"/>
@@ -82,40 +128,54 @@
   </joint>
   <link name="gripper_base">
+    <xacro:simple_inertial mass="1.5"/>
     <visual>
-      <origin xyz="0 0 0.1" rpy="0 0 0"/>
-      <geometry><box size="0.2 3 0.2"/></geometry>
+      <origin xyz="0 0 0.01" rpy="0 0 0"/>
+      <geometry><box size="0.02 0.3 0.02"/></geometry>
       <material name="grey"/>
     </visual>
+    <collision>
+      <origin xyz="0 0 0.01" rpy="0 0 0"/>
+      <geometry><box size="0.02 0.3 0.02"/></geometry>
+      <self_collide>true</self_collide>
+    </collision>
   </link>
-  <!-- Left Finger -->
+  <!--  LEFT FINGER  -->
   <joint name="finger_left_joint" type="prismatic">
     <parent link="gripper_base"/>
     <child link="gripper_finger_left"/>
-    <origin xyz="0 1.0 0.3" rpy="0 0 0"/>
+    <origin xyz="0 0.10 0.03" rpy="0 0 0"/>
     <axis xyz="0 1 0"/>
-    <limit lower="-0.9" upper="0.5" effort="10.0" velocity="0.5"/>
+    <limit lower="-0.09" upper="0.05" effort="10.0" velocity="0.5"/>
   </joint>
   <link name="gripper_finger_left">
+    <xacro:simple_inertial mass="0.3"/>
     <visual>
-      <origin xyz="0 0 0" rpy="0 0 0"/>
-      <geometry><box size="0.1 0.1 0.4"/></geometry>
+      <geometry><box size="0.01 0.01 0.04"/></geometry>
       <material name="blue"/>
     </visual>
+    <collision>
+      <geometry><box size="0.01 0.01 0.04"/></geometry>
+      <self_collide>true</self_collide>
+    </collision>
   </link>
-  <!-- Right Finger -->
+  <!--  RIGHT FINGER -->
   <joint name="finger_right_joint" type="prismatic">
     <parent link="gripper_base"/>
     <child link="gripper_finger_right"/>
-    <origin xyz="0 -1.0 0.3" rpy="0 0 0"/>
+    <origin xyz="0 -0.10 0.03" rpy="0 0 0"/>
     <axis xyz="0 -1 0"/>
-    <limit lower="-1.0" upper="0.5" effort="10.0" velocity="0.5"/>
+    <limit lower="-0.09" upper="0.05" effort="10.0" velocity="0.5"/>
     <mimic joint="finger_left_joint" multiplier="1.0" offset="0.0"/>
   </joint>
   <link name="gripper_finger_right">
+    <xacro:simple_inertial mass="0.3"/>
     <visual>
-      <origin xyz="0 0 0" rpy="0 0 0"/>
-      <geometry><box size="0.1 0.1 0.4"/></geometry>
+      <geometry><box size="0.01 0.01 0.04"/></geometry>
       <material name="blue"/>
     </visual>
+    <collision>
+      <geometry><box size="0.01 0.01 0.04"/></geometry>
+      <self_collide>true</self_collide>
+    </collision>
   </link>
 </robot>
