Commit message: fixed ratios for the hand

File: src/robocon_description/models/rrr_robot/rrr_robot.urdf (robot description, URDF)
Before this commit: robot rrr_robot, 8 links, 7 joints
Links:
- link gripper_base: geometry collision box size=0.02 0.4 0.02; visual box size=0.02 0.4 0.02
- link link3: geometry collision cylinder length=0.35 radius=0.02; visual cylinder length=0.35 radius=0.02
Joints:
- joint joint4: origin xyz=0 0 0.55 rpy=0 0 0 -> xyz=0 0 0.35 rpy=0 0 0

File: src/robocon_description/models/rrr_robot/rrr_robot.urdf.xacro (robot description, xacro)
@@ -5,5 +5,5 @@
   <xacro:property name="link1_len" value="0.27"/>
   <xacro:property name="link2_len" value="0.27"/>
-  <xacro:property name="link3_len" value="0.55"/>
+  <xacro:property name="link3_len" value="0.35"/>
   <xacro:property name="link_rad" value="0.02"/>
   <!--  MATERIALS -->
@@ -131,10 +131,10 @@
     <visual>
       <origin xyz="0 0 0.01" rpy="0 0 0"/>
-      <geometry><box size="0.02 0.3 0.02"/></geometry>
+      <geometry><box size="0.02 0.4 0.02"/></geometry>
       <material name="grey"/>
     </visual>
     <collision>
       <origin xyz="0 0 0.01" rpy="0 0 0"/>
-      <geometry><box size="0.02 0.3 0.02"/></geometry>
+      <geometry><box size="0.02 0.4 0.02"/></geometry>
       <self_collide>true</self_collide>
     </collision>

Commit message: place holder weight

File: src/robocon_description/models/rrr_robot/rrr_robot.urdf (robot description, URDF)
Before this commit: robot rrr_robot, 8 links, 7 joints
Links:
- link base_link: mass 5.0 -> 0.001
- link gripper_base: mass 1.5 -> 0.1
- link gripper_finger_left: mass 0.3 -> 0.01
- link gripper_finger_right: mass 0.3 -> 0.01
- link link0: mass 3.0 -> 0.3
- link link1: mass 4.0 -> 0.2
- link link2: mass 3.5 -> 0.3
- link link3: mass 2.5 -> 0.3

File: src/robocon_description/models/rrr_robot/rrr_robot.urdf.xacro (robot description, xacro)
@@ -25,5 +25,5 @@
   <!-- BASE -->
   <link name="base_link">
-    <xacro:simple_inertial mass="5.0"/>
+    <xacro:simple_inertial mass="0.001"/>
     <visual>
       <geometry><cylinder length="0.05" radius="0.01"/></geometry>
@@ -44,5 +44,5 @@
   <!--  LINK 0 -->
   <link name="link0">
-    <xacro:simple_inertial mass="3.0"/>
+    <xacro:simple_inertial mass="0.3"/>
     <visual>
       <origin xyz="0 0 ${link0_len/2}" rpy="0 0 0"/>
@@ -65,5 +65,5 @@
   <!-- LINK 1 -->
   <link name="link1">
-    <xacro:simple_inertial mass="4.0"/>
+    <xacro:simple_inertial mass="0.2"/>
     <visual>
       <origin xyz="0 0 ${link1_len/2}" rpy="0 0 0"/>
@@ -86,5 +86,5 @@
   <!--  LINK 2 -->
   <link name="link2">
-    <xacro:simple_inertial mass="3.5"/>
+    <xacro:simple_inertial mass="0.3"/>
     <visual>
       <origin xyz="0 0 ${link2_len/2}" rpy="0 0 0"/>
@@ -107,5 +107,5 @@
   <!--  LINK 3 -->
   <link name="link3">
-    <xacro:simple_inertial mass="2.5"/>
+    <xacro:simple_inertial mass="0.3"/>
     <visual>
       <origin xyz="0 0 ${link3_len/2}" rpy="0 0 0"/>
@@ -128,5 +128,5 @@
   </joint>
   <link name="gripper_base">
-    <xacro:simple_inertial mass="1.5"/>
+    <xacro:simple_inertial mass="0.1"/>
     <visual>
       <origin xyz="0 0 0.01" rpy="0 0 0"/>
@@ -149,5 +149,5 @@
   </joint>
   <link name="gripper_finger_left">
-    <xacro:simple_inertial mass="0.3"/>
+    <xacro:simple_inertial mass="0.01"/>
     <visual>
       <geometry><box size="0.01 0.01 0.04"/></geometry>
@@ -169,5 +169,5 @@
   </joint>
   <link name="gripper_finger_right">
-    <xacro:simple_inertial mass="0.3"/>
+    <xacro:simple_inertial mass="0.01"/>
     <visual>
       <geometry><box size="0.01 0.01 0.04"/></geometry>
