Commit message: fixing the hand rotation errror that hand is upside down

File: src/robocon_description/models/R1/urdf/hand.xacro (robot description, xacro)
@@ -133,5 +133,5 @@
       </inertial>
     </link>
-    <joint name="Revolute 1" type="revolute">
+    <joint name="revolute_1" type="revolute">
       <parent link="arm_shoulder"/>
       <child link="arm_link_1"/>
@@ -199,5 +199,5 @@
       </inertial>
     </link>
-    <joint name="Revolute 2" type="revolute">
+    <joint name="revolute_2" type="revolute">
       <parent link="arm_link_2"/>
       <child link="arm_link_2b"/>
@@ -264,5 +264,5 @@
       </inertial>
     </link>
-    <joint name="Revolute 3" type="revolute">
+    <joint name="revolute_3" type="revolute">
       <parent link="arm_link_3"/>
       <child link="arm_link_4"/>
@@ -301,5 +301,5 @@
       <parent link="arm_link_4"/>
       <child link="end_effector_link"/>
-      <origin xyz="0 0 0" rpy="0 0 0"/>
+      <origin xyz="0 0 0" rpy="3.14159 0 0"/>
     </joint>
     <!-- ======================================================== -->
@@ -328,5 +328,5 @@
       </inertial>
     </link>
-    <joint name="Revolute 4" type="revolute">
+    <joint name="revolute_4" type="revolute">
       <parent link="end_effector_link"/>
       <child link="end_effector_tip"/>
@@ -361,5 +361,5 @@
       </inertial>
     </link>
-    <joint name="Slider 1" type="prismatic">
+    <joint name="slider_1" type="prismatic">
       <parent link="end_effector_tip"/>
       <child link="right_gripper_link"/>
@@ -391,5 +391,5 @@
       </inertial>
     </link>
-    <joint name="Slider 2" type="prismatic">
+    <joint name="slider_2" type="prismatic">
       <parent link="end_effector_tip"/>
       <child link="left_gripper_link"/>
@@ -398,5 +398,5 @@
       <limit lower="-0.01280" upper="0.15775" effort="30" velocity="100"/>
       <dynamics damping="0.0" friction="0.0"/>
-      <mimic joint="Revolute 4" multiplier="1.0"/>
+      <mimic joint="slider_1" multiplier="1.0"/>
     </joint>
   </xacro:macro>

File: src/robocon_description/models/R1/urdf/robot_R1.urdf.xacro (robot description, xacro)
@@ -33,5 +33,5 @@
     <parent link="base_link_torso_mount_point"/>
     <child link="hand_root_link"/>
-    <origin xyz="0 0 0" rpy="0 0 0"/>
+    <origin xyz="0 0 0" rpy="3.14159 0 0"/>
   </joint>
 </robot>
