Commit message: fixed tf's, renamed r1 urdf better and pinkpony added nav to it to hint for navigation and changed wheels r1 to continuous. Till, Rviz, sensors spawning without errors! Except mimic.

File: src/robocon_description/models/R1/urdf/r1.urdf.xacro (robot description, xacro)
@@ -22,7 +22,7 @@
 <robot name="robot_R1" xmlns:xacro="http://ros.org/wiki/xacro">
   <!-- Include the base robot (chassis, wheels, sensors) -->
-  <xacro:include filename="base_R1.xacro" />
+  <xacro:include filename="r1_base.xacro" />
   <!-- Include the hand/arm manipulator -->
-  <xacro:include filename="hand.xacro" />
+  <xacro:include filename="r1_arm.xacro" />
   <!-- Instantiate the base -->
   <xacro:r1_base />

File: src/robocon_description/models/R1/urdf/r1_base.xacro (robot description, xacro)
@@ -71,9 +71,10 @@
     </link>
     <!-- Wheel joint -->
-    <joint name="${name}_joint" type="fixed">
+    <joint name="${name}_joint" type="continuous">
       <parent link="${motor_name}"/>
       <child link="${name}"/>
       <origin xyz="${wheel_x} ${wheel_y} ${wheel_z}"
               rpy="${wheel_roll} ${wheel_pitch} ${wheel_yaw}"/>
+      <axis xyz="0 0 1"/>
     </joint>
   </xacro:macro>
@@ -155,5 +156,6 @@
       <child link="base_link_torso_mount_point"/>
       <!-- Arm is included at this offset in R1 robot.sdf -->
-      <origin xyz="-0.239995 -0.224112 0.576396" rpy="0 0 0"/>
+      <!-- Y and Z negated to compensate for chassis_link's π-rotation around X -->
+      <origin xyz="-0.239995 0.224112 -0.576396" rpy="0 0 0"/>
     </joint>
     <!-- ============================================================ -->
